File: L2/sistabossen/sistabossen.kicad_pcb (KiCad board)
At the start: 2 copper layers, 53 x 45 mm, 22 parts, among them J1 Conn_01x02, J2 Conn_01x02, J3 Conn_01x02, J4 Conn_01x02, J5 Conn_01x02, J6 Conn_01x02, U1 TPS5430DDA

Commit message: yesbox
Parts:
- added TP1: TestPoint, TestPoint:TestPoint_THTPad_2.5x2.5mm_Drill1.2mm, F.Cu at (116.5, 53.0)
- added TP3: TestPoint, TestPoint:TestPoint_THTPad_2.5x2.5mm_Drill1.2mm, F.Cu at (70.5, 58.0)
- moved C3 1.00 mm to (83.0, 71.7)
- moved C1 0.25 mm to (111.0, 58.5)
- moved C4 0.25 mm to (115.5, 58.4)
- turned R1 to 180 degrees
Routing:
- net /PH: track 0.00 -> 52.1 mm
- net /VOUT: track 0.00 -> 42.2 mm
- net GND: track 0.00 -> 40.1 mm, vias 0 -> 4
- net /VIN: track 0.00 -> 28.4 mm
- net Net-(J3-Pin_1): track 0.00 -> 22.4 mm
- net Net-(U1-BOOT): track 0.00 -> 3.77 mm
- net Net-(J6-Pin_2): track 0.00 -> 3.46 mm
- net Net-(J5-Pin_2): track 0.00 -> 3.46 mm
- net Net-(J4-Pin_2): track 0.00 -> 3.46 mm
- net Net-(J3-Pin_2): track 0.00 -> 3.46 mm
- added copper zone on B.Cu, net GND
