File: L2/sistabossen/sistabossen.kicad_pcb (KiCad board)
At the start: 2 copper layers, 53 x 45 mm, 24 parts, among them J1 Conn_01x02, J2 Conn_01x02, J3 Conn_01x02, J4 Conn_01x02, J5 Conn_01x02, J6 Conn_01x02, U1 TPS5430DDA

Commit message: version 1.1
Parts:
- removed J6: Conn_01x02, Connector_PinHeader_2.54mm:PinHeader_1x02_P2.54mm_Vertical
- R2: value 3.24k -> 3.8k
- R3: value 5.9k -> 8.2k
- R4: value 9.53k -> 17.1k
- moved TP3 0.85 mm to (71.3, 58.3)
Connections:
- R5 pad 1: Net-(J6-Pin_2) -> Net-(J3-Pin_1)
Routing:
- net /PH: track 52.1 -> 0.00 mm
- net /VOUT: track 42.2 -> 0.14 mm
- net GND: track 40.1 -> 22.3 mm
- net /VIN: track 28.4 -> 12.8 mm
- net Net-(J3-Pin_1): track 22.4 -> 27.5 mm
- net Net-(J6-Pin_2): track 3.46 -> 0.00 mm
- added copper zone on F.Cu, net /PH
- added copper zone on F.Cu, net /VIN
- added copper zone on F.Cu, net /VOUT
- added copper zone on F.Cu, net GND
Other:
- board text added: "KTH Viktor B 2023 Djurgårdens IF"
