File: L2/sistabossen/sistabossen.kicad_pcb (KiCad board)
At the start: 2 copper layers, 53 x 45 mm, 23 parts, among them J1 Conn_01x02, J2 Conn_01x02, J3 Conn_01x02, J4 Conn_01x02, J5 Conn_01x02, U1 TPS5430DDA

Commit message: sista!!!
Parts:
- added J6: Conn_01x02, Connector_PinHeader_2.54mm:PinHeader_1x02_P2.54mm_Vertical, F.Cu at (83.0, 42.2)
Connections:
- U1 pad 5: unconnected-(U1-EN-Pad5) -> Net-(J6-Pin_2)
Routing:
- net Net-(J6-Pin_2): track 0.00 -> 42.7 mm, vias 0 -> 1
- net GND: track 22.3 -> 26.5 mm, vias 4 -> 5
Changed lines of the file:
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@@
   (net 10 "unconnected-(U1-NC-Pad2)")
   (net 11 "unconnected-(U1-NC-Pad3)")
-  (net 12 "unconnected-(U1-EN-Pad5)")
+  (net 12 "Net-(J6-Pin_2)")
   (footprint "Package_SO:TI_SO-PowerPAD-8_ThermalVias" (layer "F.Cu")
     (at 101.9 57.997056)
@@
       (net 6 "Net-(J3-Pin_1)") (pinfunction "VSENSE") (pintype "input"))
     (pad "5" smd rect (at 2.7 1.905) (size 1.55 0.6) (layers "F.Cu" "F.Paste" "F.Mask")
-      (net 12 "unconnected-(U1-EN-Pad5)") (pinfunction "EN") (pintype "input+no_connect"))
+      (net 12 "Net-(J6-Pin_2)") (pinfunction "EN") (pintype "input"))
     (pad "6" smd rect (at 2.7 0.635) (size 1.55 0.6) (layers "F.Cu" "F.Paste" "F.Mask")
       (net 2 "GND") (pinfunction "GND") (pintype "power_in"))
@@
     )
   )
+  (footprint "Connector_PinHeader_2.54mm:PinHeader_1x02_P2.54mm_Vertical" (layer "F.Cu")
+    (at 82.96 42.25 90)
+    (descr "Through hole straight pin header, 1x02, 2.54mm pitch, single row")
+    (tags "Through hole pin header THT 1x02 2.54mm single row")
+    (property "Sheetfile" "sistabossen.kicad_sch")
+    (property "Sheetname" "")
+    (property "ki_description" "Generic connector, single row, 01x02, script generated (kicad-library-utils/schlib/autogen/connector/)")
+    (property "ki_keywords" "connector")
+    (attr through_hole)
+    (fp_text reference "J6" (at 0 -2.33 90) (layer "F.SilkS")
+        (effects (font (size 1 1) (thickness 0.15)))
+    )
+    (fp_text value "Conn_01x02" (at 0 4.87 90) (layer "F.Fab")
+        (effects (font (size 1 1) (thickness 0.15)))
+    )
+    (fp_text user "${REFERENCE}" (at 0 1.27) (layer "F.Fab")
+        (effects (font (size 1 1) (thickness 0.15)))
+    )
+    (fp_line (start -1.33 -1.33) (end 0 -1.33)
+      (stroke (width 0.12) (type solid)) (layer "F.SilkS"))
+    (fp_line (start -1.33 0) (end -1.33 -1.33)
+      (stroke (width 0.12) (type solid)) (layer "F.SilkS"))
+    (fp_line (start -1.33 1.27) (end -1.33 3.87)
+      (stroke (width 0.12) (type solid)) (layer "F.SilkS"))
+    (fp_line (start -1.33 1.27) (end 1.33 1.27)
+      (stroke (width 0.12) (type solid)) (layer "F.SilkS"))
+    (fp_line (start -1.33 3.87) (end 1.33 3.87)
+      (stroke (width 0.12) (type solid)) (layer "F.SilkS"))
+    (fp_line (start 1.33 1.27) (end 1.33 3.87)
+      (stroke (width 0.12) (type solid)) (layer "F.SilkS"))
+    (fp_line (start -1.8 -1.8) (end -1.8 4.35)
+      (stroke (width 0.05) (type solid)) (layer "F.CrtYd"))
+    (fp_line (start -1.8 4.35) (end 1.8 4.35)
+      (stroke (width 0.05) (type solid)) (layer "F.CrtYd"))
+    (fp_line (start 1.8 -1.8) (end -1.8 -1.8)
+      (stroke (width 0.05) (type solid)) (layer "F.CrtYd"))
+    (fp_line (start 1.8 4.35) (end 1.8 -1.8)
+      (stroke (width 0.05) (type solid)) (layer "F.CrtYd"))
+    (fp_line (start -1.27 -0.635) (end -0.635 -1.27)
+      (stroke (width 0.1) (type solid)) (layer "F.Fab"))
+    (fp_line (start -1.27 3.81) (end -1.27 -0.635)
+      (stroke (width 0.1) (type solid)) (layer "F.Fab"))
+    (fp_line (start -0.635 -1.27) (end 1.27 -1.27)
+      (stroke (width 0.1) (type solid)) (layer "F.Fab"))
+    (fp_line (start 1.27 -1.27) (end 1.27 3.81)
+      (stroke (width 0.1) (type solid)) (layer "F.Fab"))
+    (fp_line (start 1.27 3.81) (end -1.27 3.81)
+      (stroke (width 0.1) (type solid)) (layer "F.Fab"))
+    (pad "1" thru_hole rect (at 0 0 90) (size 1.7 1.7) (drill 1) (layers "*.Cu" "*.Mask")
+      (net 2 "GND") (pinfunction "Pin_1") (pintype "passive"))
+    (pad "2" thru_hole oval (at 0 2.54 90) (size 1.7 1.7) (drill 1) (layers "*.Cu" "*.Mask")
+      (net 12 "Net-(J6-Pin_2)") (pinfunction "Pin_2") (pintype "passive"))
+    (model "${KICAD6_3DMODEL_DIR}/Connector_PinHeader_2.54mm.3dshapes/PinHeader_1x02_P2.54mm_Vertical.wrl"
+      (offset (xyz 0 0 0))
+      (scale (xyz 1 1 1))
+      (rotate (xyz 0 0 0))
+    )
+  )
   (footprint "Capacitor_SMD:C_0805_2012Metric_Pad1.18x1.45mm_HandSolder" (layer "F.Cu")
     (at 115.5 58.4125 -90)
@@
   (segment (start 111 59.4875) (end 111 61) (width 0.25) (layer "F.Cu") (net 2))
   (segment (start 111.0375 59.45) (end 111 59.4875) (width 0.25) (layer "F.Cu") (net 2))
+  (segment (start 82.96 42.25) (end 78.75 42.25) (width 0.25) (layer "F.Cu") (net 2))
   (segment (start 102.5 58.697056) (end 101.3 58.697056) (width 0.25) (layer "F.Cu") (net 2))
   (segment (start 111 59.4875) (end 110.9875 59.5) (width 0.25) (layer "F.Cu") (net 2))
@@
   (segment (start 107.632056 58.632056) (end 104.6 58.632056) (width 0.25) (layer "F.Cu") (net 2))
   (via (at 101 80.5) (size 0.8) (drill 0.4) (layers "F.Cu" "B.Cu") (free) (net 2))
+  (via (at 78.75 42.25) (size 0.8) (drill 0.4) (layers "F.Cu" "B.Cu") (free) (net 2))
   (via (at 111 61) (size 0.8) (drill 0.4) (layers "F.Cu" "B.Cu") (free) (net 2))
   (via (at 101 49.5) (size 0.8) (drill 0.4) (layers "F.Cu" "B.Cu") (net 2))
@@
   (segment (start 98.96 69.697056) (end 95.5 69.697056) (width 0.25) (layer "F.Cu") (net 8))
   (segment (start 98.96 73.697056) (end 95.5 73.697056) (width 0.25) (layer "F.Cu") (net 9))
+  (segment (start 104.6 59.902056) (end 106.902056 59.902056) (width 0.25) (layer "F.Cu") (net 12))
+  (segment (start 106.902056 59.902056) (end 107.25 60.25) (width 0.25) (layer "F.Cu") (net 12))
+  (via (at 107.25 60.25) (size 0.8) (drill 0.4) (layers "F.Cu" "B.Cu") (free) (net 12))
+  (segment (start 92 62.75) (end 105.5 62.75) (width 0.25) (layer "B.Cu") (net 12))
+  (segment (start 85.5 42.25) (end 85.5 56.25) (width 0.25) (layer "B.Cu") (net 12))
+  (segment (start 85.5 56.25) (end 92 62.75) (width 0.25) (layer "B.Cu") (net 12))
+  (segment (start 105.5 62.75) (end 107.25 61) (width 0.25) (layer "B.Cu") (net 12))
+  (segment (start 107.25 61) (end 107.25 60.25) (width 0.25) (layer "B.Cu") (net 12))
   (zone (net 5) (net_name "/VOUT") (layer "F.Cu") (hatch edge 0.5)
     (priority 3)
