File: L2/sistabossen/sistabossen.kicad_sch (KiCad schematic)
At the start: 22 parts, among them J1 Conn_01x02, J2 Conn_01x02, J3 Conn_01x02, J4 Conn_01x02, J5 Conn_01x02, J6 Conn_01x02, U1 TPS5430DDA

Commit message: yesbox
Parts:
- added TP1, TP3: TestPoint, TestPoint:TestPoint_THTPad_2.5x2.5mm_Drill1.2mm, symbol Connector:TestPoint
Connections:
- net VIN: now also TP1.1
- net VOUT: now also TP3.1
Changed lines of the file:
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@@
+    (stroke (width 0) (type default))
+  )
+  (wire (pts (xy 90.17 64.77) (xy 87.63 64.77))
+    (stroke (width 0) (type default))
+  )
+  (wire (pts (xy 193.04 67.31) (xy 193.04 71.12))
+    (stroke (width 0) (type default))
+  )
+  (wire (pts (xy 172.72 73.66) (xy 172.72 78.74))
+    (stroke (width 0) (type default))
+  )
+  (wire (pts (xy 54.61 46.99) (xy 64.77 46.99))
+    (stroke (width 0) (type default))
+  )
+  (wire (pts (xy 162.56 59.69) (xy 162.56 60.96))
     (stroke (width 0) (type default))
   )
@@
     (stroke (width 0) (type default))
   )
-  (wire (pts (xy 90.17 64.77) (xy 87.63 64.77))
-    (stroke (width 0) (type default))
-  )
-  (wire (pts (xy 193.04 67.31) (xy 193.04 71.12))
-    (stroke (width 0) (type default))
-  )
-  (wire (pts (xy 172.72 73.66) (xy 172.72 78.74))
-    (stroke (width 0) (type default))
-  )
-  (wire (pts (xy 54.61 46.99) (xy 64.77 46.99))
-    (stroke (width 0) (type default))
-  )
-  (wire (pts (xy 162.56 59.69) (xy 162.56 60.96))
-    (stroke (width 0) (type default))
-  )
   (wire (pts (xy 90.17 62.23) (xy 90.17 64.77))
     (stroke (width 0) (type default))
@@
     (stroke (width 0) (type default))
   )
+  (wire (pts (xy 45.72 46.99) (xy 54.61 46.99))
+    (stroke (width 0) (type default))
+  )
   (wire (pts (xy 193.04 86.36) (xy 193.04 87.63))
     (stroke (width 0) (type default))
@@
     (stroke (width 0) (type default))
   )
+  (wire (pts (xy 162.56 46.99) (xy 171.45 46.99))
+    (stroke (width 0) (type default))
+  )
   (wire (pts (xy 116.84 46.99) (xy 121.92 46.99))
     (stroke (width 0) (type default))
@@
     (stroke (width 0) (type default))
   )
-  (wire (pts (xy 162.56 46.99) (xy 171.45 46.99))
-    (stroke (width 0) (type default))
-  )
   (wire (pts (xy 64.77 46.99) (xy 74.93 46.99))
-    (stroke (width 0) (type default))
-  )
-  (wire (pts (xy 45.72 46.99) (xy 54.61 46.99))
     (stroke (width 0) (type default))
   )
@@
     )
   )
+  (symbol (lib_id "Connector:TestPoint") (at 54.61 46.99 0) (unit 1)
+    (in_bom yes) (on_board yes) (dnp no) (fields_autoplaced)
+    (property "Reference" "TP1" (at 57.15 43.053 0)
+      (effects (font (size 1.27 1.27)) (justify left))
+    )
+    (property "Value" "TestPoint" (at 57.15 45.593 0)
+      (effects (font (size 1.27 1.27)) (justify left))
+    )
+    (property "Footprint" "TestPoint:TestPoint_THTPad_2.5x2.5mm_Drill1.2mm" (at 59.69 46.99 0)
+      (effects (font (size 1.27 1.27)) hide)
+    )
+    (property "Datasheet" "~" (at 59.69 46.99 0)
+      (effects (font (size 1.27 1.27)) hide)
+    )
+    (pin "1")
+    (instances
+      (project "sistabossen"
+        (path "/07dfce2c-367d-460b-a7d9-6de3122686da"
+          (reference "TP1") (unit 1)
+        )
+      )
+    )
+  )
   (symbol (lib_id "Mechanical:MountingHole_Pad") (at 78.74 120.65 0) (unit 1)
     (in_bom yes) (on_board yes) (dnp no) (fields_autoplaced)
@@
         )
       )
+    )
+  )
+  (symbol (lib_id "Connector:TestPoint") (at 162.56 46.99 0) (unit 1)
+    (in_bom yes) (on_board yes) (dnp no) (fields_autoplaced)
+    (property "Reference" "TP3" (at 165.1 43.053 0)
+      (effects (font (size 1.27 1.27)) (justify left))
+    )
+    (property "Value" "TestPoint" (at 165.1 45.593 0)
+      (effects (font (size 1.27 1.27)) (justify left))
+    )
+    (property "Footprint" "TestPoint:TestPoint_THTPad_2.5x2.5mm_Drill1.2mm" (at 167.64 46.99 0)
+      (effects (font (size 1.27 1.27)) hide)
+    )
+    (property "Datasheet" "~" (at 167.64 46.99 0)
+      (effects (font (size 1.27 1.27)) hide)
+    )
+    (pin "1")
+    (instances
+      (project "sistabossen"
+        (path "/07dfce2c-367d-460b-a7d9-6de3122686da"
+          (reference "TP3") (unit 1)
+        )
+      )

Commit message: version 1.1
Parts:
- removed J6: Conn_01x02, Connector_PinHeader_2.54mm:PinHeader_1x02_P2.54mm_Vertical, symbol Connector_Generic:Conn_01x02
- R2: value 3.24k -> 3.8k
- R3: value 5.9k -> 8.2k
- R4: value 9.53k -> 17.1k
Connections:
- net at J3.1 (Pin_1), J4.1 (Pin_1), J5.1 (Pin_1)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: now also R5.1
Changed lines of the file:
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@@
     (stroke (width 0) (type default))
   )
-  (wire (pts (xy 193.04 67.31) (xy 193.04 71.12))
+  (wire (pts (xy 193.04 67.31) (xy 193.04 78.74))
     (stroke (width 0) (type default))
   )
@@
   )
   (wire (pts (xy 172.72 67.31) (xy 182.88 67.31))
-    (stroke (width 0) (type default))
-  )
-  (wire (pts (xy 193.04 73.66) (xy 193.04 78.74))
     (stroke (width 0) (type default))
   )
@@
       (effects (font (size 1.27 1.27)) (justify left))
     )
-    (property "Value" "3.24k" (at 165.1 84.455 0)
+    (property "Value" "3.8k" (at 165.1 84.455 0)
       (effects (font (size 1.27 1.27)) (justify left))
     )
@@
       (effects (font (size 1.27 1.27)) (justify left))
     )
-    (property "Value" "9.53k" (at 185.42 84.455 0)
+    (property "Value" "17.1k" (at 185.42 84.455 0)
       (effects (font (size 1.27 1.27)) (justify left))
     )
@@
         (path "/07dfce2c-367d-460b-a7d9-6de3122686da"
           (reference "J2") (unit 1)
-        )
-      )
-    )
-  )
-  (symbol (lib_id "Connector_Generic:Conn_01x02") (at 198.12 71.12 0) (unit 1)
-    (in_bom yes) (on_board yes) (dnp no) (fields_autoplaced)
-    (property "Reference" "J6" (at 200.66 71.755 0)
-      (effects (font (size 1.27 1.27)) (justify left))
-    )
-    (property "Value" "Conn_01x02" (at 200.66 74.295 0)
-      (effects (font (size 1.27 1.27)) (justify left) hide)
-    )
-    (property "Footprint" "Connector_PinHeader_2.54mm:PinHeader_1x02_P2.54mm_Vertical" (at 198.12 71.12 0)
-      (effects (font (size 1.27 1.27)) hide)
-    )
-    (property "Datasheet" "~" (at 198.12 71.12 0)
-      (effects (font (size 1.27 1.27)) hide)
-    )
-    (pin "1")
-    (pin "2")
-    (instances
-      (project "sistabossen"
-        (path "/07dfce2c-367d-460b-a7d9-6de3122686da"
-          (reference "J6") (unit 1)
         )
       )
@@
       (effects (font (size 1.27 1.27)) (justify left))
     )
-    (property "Value" "5.9k" (at 175.26 84.455 0)
-      (effects (font (size 1.27 1.27)) (justify left))
-    )
+    (property "Value" "8.2k" (at 175.26 84.455 0)
+      (effects (font (size 1.27 1.27)) (justify left))
+    )

Commit message: sista!!!
Parts:
- added J6: Conn_01x02, Connector_PinHeader_2.54mm:PinHeader_1x02_P2.54mm_Vertical, symbol Connector_Generic:Conn_01x02
Connections:
- net GND: now also J6.1 (Pin_1)
- net at U1.5 (EN): now also J6.2 (Pin_2)
- no-connect marks 1 -> 0
Changed lines of the file:
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@@
   (junction (at 162.56 60.96) (diameter 0) (color 0 0 0 0)
   )
-  (no_connect (at 77.47 57.15))
   (wire (pts (xy 102.87 57.15) (xy 116.84 57.15))
     (stroke (width 0) (type default))
@@
     (stroke (width 0) (type default))
   )
+  (wire (pts (xy 74.93 57.15) (xy 74.93 62.23))
+    (stroke (width 0) (type default))
+  )
   (wire (pts (xy 58.42 123.19) (xy 58.42 125.73))
     (stroke (width 0) (type default))
@@
     (stroke (width 0) (type default))
   )
+  (wire (pts (xy 74.93 64.77) (xy 74.93 71.12))
+    (stroke (width 0) (type default))
+  )
   (wire (pts (xy 162.56 86.36) (xy 162.56 87.63))
     (stroke (width 0) (type default))
@@
   )
   (wire (pts (xy 121.92 59.69) (xy 121.92 71.12))
+    (stroke (width 0) (type default))
+  )
+  (wire (pts (xy 77.47 57.15) (xy 74.93 57.15))
     (stroke (width 0) (type default))
   )
@@
     )
   )
+  (symbol (lib_id "Connector_Generic:Conn_01x02") (at 69.85 64.77 180) (unit 1)
+    (in_bom yes) (on_board yes) (dnp no) (fields_autoplaced)
+    (property "Reference" "J6" (at 69.85 59.69 0)
+      (effects (font (size 1.27 1.27)))
+    )
+    (property "Value" "Conn_01x02" (at 67.31 61.595 0)
+      (effects (font (size 1.27 1.27)) (justify left) hide)
+    )
+    (property "Footprint" "Connector_PinHeader_2.54mm:PinHeader_1x02_P2.54mm_Vertical" (at 69.85 64.77 0)
+      (effects (font (size 1.27 1.27)) hide)
+    )
+    (property "Datasheet" "~" (at 69.85 64.77 0)
+      (effects (font (size 1.27 1.27)) hide)
+    )
+    (pin "1")
+    (pin "2")
+    (instances
+      (project "sistabossen"
+        (path "/07dfce2c-367d-460b-a7d9-6de3122686da"
+          (reference "J6") (unit 1)
+        )
+      )
+    )
+  )
   (symbol (lib_id "power:GND") (at 48.26 125.73 0) (unit 1)
     (in_bom yes) (on_board yes) (dnp no) (fields_autoplaced)
@@
         )
       )
+    )
+  )
+  (symbol (lib_id "power:GND") (at 74.93 71.12 0) (unit 1)
+    (in_bom yes) (on_board yes) (dnp no) (fields_autoplaced)
+    (property "Reference" "#PWR016" (at 74.93 77.47 0)
+      (effects (font (size 1.27 1.27)) hide)
+    )
+    (property "Value" "GND" (at 74.93 76.2 0)
+      (effects (font (size 1.27 1.27)))
+    )
+    (property "Footprint" "" (at 74.93 71.12 0)
+      (effects (font (size 1.27 1.27)) hide)
+    )
+    (property "Datasheet" "" (at 74.93 71.12 0)
+      (effects (font (size 1.27 1.27)) hide)
+    )
+    (pin "1")
+    (instances
+      (project "sistabossen"
+        (path "/07dfce2c-367d-460b-a7d9-6de3122686da"
+          (reference "#PWR016") (unit 1)
+        )
+      )
